Commit message: making nav2 working without map and on gps

File: bumperbot_ws/install/bumperbot_description/share/bumperbot_description/urdf/bumperbot.urdf.xacro (robot description, xacro)
@@ -1,3 +1,2 @@
-<?xml version="1.0"?>
 <robot xmlns:xacro="http://www.ros.org/wiki/xacro" name="bumperbot">
     <xacro:arg name="is_sim" default="true"/>
@@ -153,4 +152,11 @@
         </collision>
     </link>
+    <link name="gps_link"/>
+    <!-- Add the gps link so we get a static transform for the GPS -->
+    <joint name="gps_joint" type="fixed">
+      <parent link="base_link"/>
+      <child link="gps_link"/>
+      <origin xyz="0 0 0" rpy="0 0 0"/>
+    </joint>
     <joint name="base_joint" type="fixed">
         <parent link="base_footprint"/>

File: bumperbot_ws/install/bumperbot_description/share/bumperbot_description/urdf/bumperbot_gazebo.xacro (robot description, xacro)
@@ -1,3 +1,2 @@
-<?xml version="1.0" encoding="UTF-8"?>
 <robot name="bumperbot" xmlns:xacro="http://www.ros.org/wiki/xacro">
     <transmission name="wheel_right_transmission">
@@ -106,4 +105,39 @@
       </sensor>
     </gazebo>
+    <gazebo reference="gps_link">
+      <spherical_coordinates>
+        <surface_model>EARTH_WGS84</surface_model>
+        <latitude_deg>38.161479</latitude_deg>
+        <longitude_deg>-122.454630</longitude_deg>
+        <elevation>488.0</elevation>
+        <heading_deg>180</heading_deg>
+      </spherical_coordinates>
+      <sensor name="tb3_gps" type="gps">
+        <always_on>true</always_on>
+        <update_rate>1</update_rate>
+        <pose>0 0 0 0 0 0</pose>
+        <gps>
+          <position_sensing>
+            <horizontal>
+              <noise type="gaussian">
+                <mean>0.0</mean>
+                <stddev>0.01</stddev>
+              </noise>
+            </horizontal>
+            <vertical>
+              <noise type="gaussian">
+                <mean>0.0</mean>
+                <stddev>0.01</stddev>
+              </noise>
+            </vertical>
+          </position_sensing>
+        </gps>
+        <plugin name="my_gps_plugin" filename="libgazebo_ros_gps_sensor.so">
+          <ros>
+            <remapping>~/out:=/gps/fix</remapping>
+          </ros>
+        </plugin>
+      </sensor>
+    </gazebo>
 <!--
     <gazebo reference="laser_link">

File: bumperbot_ws/install/bumperbot_description/share/bumperbot_description/urdf/bumperbot_ros2_control.xacro (robot description, xacro)
@@ -1,3 +1,2 @@
-<?xml version="1.0"?>
 <robot xmlns:xacro="http://www.ros.org/wiki/xacro" name="bumperbot">
     <ros2_control name="RobotSystem" type="system">
